Commit message: workcell added

File: ur_description/urdf/ur3_robot_erc.urdf.xacro (robot description, xacro)
@@ -11,4 +11,10 @@
     transmission_hw_interface="$(arg transmission_hw_interface)"
   />
+<link name="world" />
+  <joint name="world_joint" type="fixed">
+    <parent link="world" />
+    <child link = "base_link" />
+    <origin xyz="0.0 0.0 0.0" rpy="0.0 0.0 0.0" />
+  </joint>
   <link name="gripper">
     <visual>
@@ -26,5 +32,5 @@
     <inertial>
         <!-- The following are not reliable values, and should not be used for modeling -->
-        <mass value="0.5" />
+        <mass value="0.01" />
         <origin xyz="0 0 0" />
         <inertia ixx="534306880.000000" ixy="-297469.312500" ixz="-4140206.750000" iyx="-297469.312500" iyy="452308608.000000" iyz="83961360.000000" izx="-4140206.750000" izy="83961360.000000" izz="303997888.000000" />
